File: current/MRR_ESPA.kicad_pcb (KiCad board)
At the start: 2 copper layers, 99.5 x 90.5 mm, 129 parts, among them J1 X_MIN, J10 PART_FAN, J11 FAN_HEATSINK, J12 T_BED, J13 T_E0, J14 I2C/SPI, J15 AUX1, J16 USB_B_Micro, J17 CS_PINS, J2 Z_MIN, J21 X_MOTOR, J22 Z_MOTOR, J23 Y_MOTOR, J24 E0_MOTOR, J3 BED, J4 Micro_SD_Card_China, J5 Y_MIN, J6 Z_PROBE, J7 E0, J8 FAN_CASE, J9 PWR_IN, Q1 WSK220N04, Q2 WSF3085, Q3 WST3038, Q4 S9014, Q5 S9014, SW1 RESET, U1 ESP32-WROOM-32D, U10 TLP182, U11 74LVC1G125, U12 74LVC1G125, U2 TPS54340DDA, U3 CH340C, U4 AMS1117-3.3, U5 Pololu_board, U6 Pololu_board, U8 Pololu_board, U9 Pololu_board

Commit message: Added v1.3 files
Parts:
- added C28: 100nF25V, Capacitor_SMD:C_0805_2012Metric, F.Cu at (72.5, 81.8)
- C1, C2, C3: value 100nF16V -> 100nF25V
- C11: value 10nF16V -> 10nF50V
- C13, C14: value 47uF16V -> 47uF6.3V
- C19: value 100uF10V -> 100uF6.3V
- C5, C6: value 10uF16V -> 22uF6.3V
- D14, D15: value 1N5819 -> 1N5819W
- D4, D5: value 1N4007 -> 1N4007W
- F1: value 10A 1808 -> 15A 2410
- F2: value 20A 1808 -> 30A 3912; footprint projfp:Littelfuse_0451 -> projfp:Littelfuse_456
- JP17: value VUSB_EN -> 5V_SEL; footprint Connector_PinHeader_2.54mm:PinHeader_1x02_P2.54mm_Vertical -> Connector_PinHeader_2.54mm:PinHeader_1x03_P2.54mm_Vertical
- Q3: value WST3038 -> WSF3038
- moved JP17 7.09 mm to (103.3, 61.8), turned to 270 degrees
- moved R29 6.87 mm to (95.0, 65.0), turned to 90 degrees
- moved D11 5.72 mm to (92.1, 65.7)
- moved D14 3.49 mm to (103.7, 56.9), turned to 0 degrees
- moved D15 3.12 mm to (98.7, 56.9), turned to 0 degrees
- moved F2 2.97 mm to (124.7, 85.8)
- moved J10 1.95 mm to (142.6, 113.7)
- moved D1 1.01 mm to (120.4, 89.6)
- moved R5 0.23 mm to (121.3, 85.9)
- moved C14 0.09 mm to (102.2, 67.8)
Connections:
- D14 pad 1: +5V -> Net-(D14-Pad1)
- D15 pad 1: +5V -> Net-(D15-Pad1)
- D15 pad 2: Net-(D15-Pad2) -> VUSB
- JP17 pad 1: Net-(D15-Pad2) -> Net-(D14-Pad1)
- JP17 pad 2: VUSB -> +5V
Routing:
- net Net-(D15-Pad1): track 0.00 -> 5.23 mm
- net Net-(D14-Pad1): track 0.00 -> 5.12 mm
- net VIN: track 380.8 -> 377.8 mm
- net Net-(D15-Pad2): track 2.71 -> 0.00 mm
- net Net-(D11-Pad2): track 4.77 -> 2.27 mm
- net VUSB: track 5.33 -> 7.82 mm
- net EN: track 45.7 -> 47.7 mm
- net +5V: track 67.5 -> 65.9 mm
- net +3V3: track 415.5 -> 417.0 mm
- net MOSI: track 191.9 -> 192.8 mm
- net Net-(D1-Pad1): track 4.21 -> 4.82 mm
- net GND: vias 82 -> 108
Other:
- board text added: "EN"
- board text added: "MRR ESPA v1.3"
- board text added: "VUSB"
- board text added: "Version date: 2019-10-06"
- board text removed: "MRR ESPA v1.2"
- board text removed: "Version date: 2019-07-06"
