File: current/MRR_ESPA.sch (KiCad schematic (older format))
At the start: 129 parts, among them J1 X_MIN, J10 PART_FAN, J11 FAN_HEATSINK, J12 T_BED, J13 T_E0, J14 I2C/SPI, J15 AUX1, J16 USB_B_Micro, J17 CS_PINS, J2 Z_MIN, J21 X_MOTOR, J22 Z_MOTOR, J23 Y_MOTOR, J24 E0_MOTOR, J3 BED, J4 Micro_SD_Card_China, J5 Y_MIN, J6 Z_PROBE, J7 E0, J8 FAN_CASE, J9 PWR_IN, Q1 WSK220N04, Q2 WSF3085, Q3 WST3038, Q4 S9014, Q5 S9014, SW1 RESET, U1 ESP32-WROOM-32D, U10 TLP182, U11 74LVC1G125, U12 74LVC1G125, U2 TPS54340DDA, U3 CH340C, U4 AMS1117-3.3, U5 Pololu_board, U6 Pololu_board, U8 Pololu_board, U9 Pololu_board

Commit message: Added v1.3 files
Parts:
- removed JP17: VUSB_EN, Connector_PinHeader_2.54mm:PinHeader_1x02_P2.54mm_Vertical, symbol Device:Jumper
- added C28: 100nF25V, Capacitor_SMD:C_0805_2012Metric, symbol Device:C
- added JP17: 5V_SEL, Connector_PinHeader_2.54mm:PinHeader_1x03_P2.54mm_Vertical, symbol Jumper:Jumper_3_Open
- C1, C2, C3: value 100nF16V -> 100nF25V; LCSC Part Number (none) -> C128353; Manufacturer (none) -> Walsin Tech Corp; Mfg part no. (none) -> 0805B104K250
- C10: LCSC Part Number (none) -> C161260; Manufacturer (none) -> Murata Electronics; Mfg part no. (none) -> GCM21BR71H104KA37L
- C11: value 10nF16V -> 10nF50V; LCSC Part Number (none) -> C52278; Manufacturer (none) -> Guangdong Fenghua Advanced Tech; Mfg part no. (none) -> 0805B103K500NT
- C12: LCSC Part Number (none) -> C92821; Manufacturer (none) -> Taiyo Yuden; Mfg part no. (none) -> LMK316BJ476ML-T
- C13, C14: value 47uF16V -> 47uF6.3V; LCSC Part Number (none) -> C87159; Manufacturer (none) -> Taiyo Yuden; Mfg part no. (none) -> JMK212BJ476MG-T
- C15, C16, C17, C18: LCSC Part Number (none) -> C97811; Manufacturer (none) -> Semtech; Mfg part no. (none) -> CS1V101M-CRE77
- C19: value 100uF10V -> 100uF6.3V; LCSC Part Number (none) -> C15008; Manufacturer (none) -> Samsung Electro-Mechanics; Mfg part no. (none) -> CL31A107MQHNNNE
- C4: LCSC Part Number (none) -> C176665; Manufacturer (none) -> Lelon; Mfg part no. (none) -> VEJ101M1HTR-0810
- C5, C6: value 10uF16V -> 22uF6.3V; LCSC Part Number (none) -> C5674; Manufacturer (none) -> Samsung Electro-Mechanics; Mfg part no. (none) -> CL21A226MQQNNNE
- C7: LCSC Part Number (none) -> C307575; Manufacturer (none) -> Samsung Electro-Mechanics; Mfg part no. (none) -> CL31B475KBHNFNE
- C8: LCSC Part Number (none) -> C152862; Manufacturer (none) -> Walsin Tech Corp; Mfg part no. (none) -> 0805B821K500CT
- C9: LCSC Part Number (none) -> C296102; Manufacturer (none) -> Walsin Tech Corp; Mfg part no. (none) -> 0805N560J500CT
- D1, D3, D6: LCSC Part Number (none) -> C72037; Manufacturer (none) -> Everlight Elec; Mfg part no. (none) -> 17-21SURC/S530-A3/TR8
- D10, D11: LCSC Part Number (none) -> C73548; Manufacturer (none) -> Everlight Elec; Mfg part no. (none) -> 17-21SYGC/S530-E2/TR8
- D12, D13: LCSC Part Number (none) -> C72035; Manufacturer (none) -> Everlight Elec; Mfg part no. (none) -> 17-21/BHC-XL2M2TY/3T
- D14, D15: value 1N5819 -> 1N5819W; LCSC Part Number (none) -> C169540; Manufacturer (none) -> Shandong Jingdao Microelectronics; Mfg part no. (none) -> 1N5819W
- D2: LCSC Part Number (none) -> C81598; Manufacturer (none) -> Semtech; Mfg part no. (none) -> 1N4148W
- D4, D5: value 1N4007 -> 1N4007W; LCSC Part Number (none) -> C108803; Manufacturer (none) -> Shandong Jingdao Microelectronics; Mfg part no. (none) -> 1N4007W
- D7, D8: LCSC Part Number (none) -> C19224; Manufacturer (none) -> Nexperia; Mfg part no. (none) -> PESD5V0S1BA,115
- D9: LCSC Part Number (none) -> C72264; Manufacturer (none) -> Diodes Incorporated; Mfg part no. (none) -> B540C-13-F
- F1: value 10A 1808 -> 15A 2410; LCSC Part Number (none) -> C44480; Manufacturer (none) -> Littelfuse; Mfg part no. (none) -> 0451015.MRL
- F2: value 20A 1808 -> 30A 3912; footprint projfp:Littelfuse_0451 -> projfp:Littelfuse_456; LCSC Part Number (none) -> C187558; Manufacturer (none) -> Littelfuse; Mfg part no. (none) -> 0456030.ER
- J1, J2, J5, J6: LCSC Part Number (none) -> C144394; Manufacturer (none) -> JST Sales America; Mfg part no. (none) -> B3B-XH-A(LF)(SN)
- J10, J11, J8: LCSC Part Number (none) -> C124375; Manufacturer (none) -> Shenzhen Cankemeng; Mfg part no. (none) -> C124375
- J12, J13: LCSC Part Number (none) -> C158012; Manufacturer (none) -> JST Sales America; Mfg part no. (none) -> B2B-XH-A(LF)(SN)
- J14: LCSC Part Number (none) -> C124381; Manufacturer (none) -> Shenzhen Cankemeng; Mfg part no. (none) -> C124381
- J15: LCSC Part Number (none) -> C9135; Manufacturer (none) -> Boom Precision Elec; Mfg part no. (none) -> C9135
- J16: LCSC Part Number (none) -> C136000; Manufacturer (none) -> MOLEX; Mfg part no. (none) -> 105017-0001
- J17, J21, J23, J24: LCSC Part Number (none) -> C124378; Manufacturer (none) -> Shenzhen Cankemeng; Mfg part no. (none) -> C124378
- J22: LCSC Part Number (none) -> C124386; Manufacturer (none) -> Shenzhen Cankemeng; Mfg part no. (none) -> C124386
- J3: LCSC Part Number (none) -> C89120; Manufacturer (none) -> Phoenix Contact; Mfg part no. (none) -> MKDS3/2-5.08
- J4: LCSC Part Number (none) -> C111196; Manufacturer (none) -> SOFNG; Mfg part no. (none) -> TF-15×15
- J7: LCSC Part Number (none) -> C91153; Manufacturer (none) -> Phoenix Contact; Mfg part no. (none) -> MKDSN1.5/2-5.08
- J9: LCSC Part Number (none) -> C90087; Manufacturer (none) -> Phoenix Contact; Mfg part no. (none) -> MKDS3/4-5.08
- JP1, JP10, JP11, JP12, JP13, JP14, JP15, JP16, JP18, JP2, JP3, JP4, JP5, JP6, JP7, JP8, JP9: LCSC Part Number (none) -> C124376; Manufacturer (none) -> Shenzhen Cankemeng; Mfg part no. (none) -> C124376
- L1: LCSC Part Number (none) -> C181722; Manufacturer (none) -> Shun Xiang Nuo Elec; Mfg part no. (none) -> SMMS0530-4R7M
- Q1: LCSC Part Number (none) -> C148446; Manufacturer (none) -> Winsok Semicon; Mfg part no. (none) -> WSK220N04
- Q2: LCSC Part Number (none) -> C148428; Manufacturer (none) -> Winsok Semicon; Mfg part no. (none) -> WSF3085
- Q3: value WST3038 -> WSF3038; LCSC Part Number (none) -> C148426; Manufacturer (none) -> Winsok Semicon; Mfg part no. (none) -> WSF3038
- Q4, Q5: LCSC Part Number (none) -> C181164; Manufacturer (none) -> Guangdong Hottech; Mfg part no. (none) -> S9014
- R1, R3, R32, R4, R8: LCSC Part Number (none) -> C38522; Manufacturer (none) -> Uniroyal Elec; Mfg part no. (none) -> 0805W8F2201T5E
- R10, R13: LCSC Part Number (none) -> C17415; Manufacturer (none) -> Uniroyal Elec; Mfg part no. (none) -> 0805W8F100JT5E
- R11, R14: LCSC Part Number (none) -> C149504; Manufacturer (none) -> Uniroyal Elec; Mfg part no. (none) -> 0805W8F1003T5E
- R12, R30, R31, R5, R9: LCSC Part Number (none) -> C17520; Manufacturer (none) -> Uniroyal Elec; Mfg part no. (none) -> 0805W8F2201T5E
- R15, R22, R23: LCSC Part Number (none) -> C17444; Manufacturer (none) -> Uniroyal Elec; Mfg part no. (none) -> 0805W8F1202T5E
- R16, R17, R19, R20: LCSC Part Number (none) -> C17673; Manufacturer (none) -> Uniroyal Elec; Mfg part no. (none) -> 0805W8F4701T5E
- R18: LCSC Part Number (none) -> C170958; Manufacturer (none) -> Walsin Tech Corp; Mfg part no. (none) -> WR08X7322FTL
- R21: LCSC Part Number (none) -> C170848; Manufacturer (none) -> Walsin Tech Corp; Mfg part no. (none) -> WR08X2372FTL
- R24: LCSC Part Number (none) -> C273994; Manufacturer (none) -> YAGEO; Mfg part no. (none) -> RC0805FR-0760K4L
- R25: LCSC Part Number (none) -> C17418; Manufacturer (none) -> Uniroyal Elec; Mfg part no. (none) -> 0805W8F1152T5E
- R26, R27: LCSC Part Number (none) -> C17477; Manufacturer (none) -> Uniroyal Elec; Mfg part no. (none) -> 0805W8F0000T5E
- R28: LCSC Part Number (none) -> C17557; Manufacturer (none) -> Uniroyal Elec; Mfg part no. (none) -> 0805W8F2200T5E
- R29, R36: LCSC Part Number (none) -> C17630; Manufacturer (none) -> Uniroyal Elec; Mfg part no. (none) -> 0805W8F3300T5E
- R35, R38: LCSC Part Number (none) -> C17513; Manufacturer (none) -> Uniroyal Elec; Mfg part no. (none) -> 0805W8F1001T5E
- SW1: LCSC Part Number (none) -> C83206; Manufacturer (none) -> Korean Hroparts Elec; Mfg part no. (none) -> K2-6639SP-C4SC-04
- U1: LCSC Part Number (none) -> C95209; Manufacturer (none) -> Espressif Systems; Mfg part no. (none) -> ESP32-WROOM-32
- U10: LCSC Part Number (none) -> C96457; Manufacturer (none) -> TOSHIBA; Mfg part no. (none) -> TLP182(GB-TPL,E
- U11, U12: LCSC Part Number (none) -> C12519; Manufacturer (none) -> Nexperia; Mfg part no. (none) -> 74LVC1G125GW,125
- U2: LCSC Part Number (none) -> C45886; Manufacturer (none) -> Texas Instruments; Mfg part no. (none) -> TPS54340DDAR
- U3: LCSC Part Number (none) -> C84681; Manufacturer (none) -> Jiangsu Qin Heng; Mfg part no. (none) -> CH340C
- U4: LCSC Part Number (none) -> C6186; Manufacturer (none) -> Advanced Monolithic Systems; Mfg part no. (none) -> AMS1117-3.3
- U5, U6, U8, U9: LCSC Part Number (none) -> C27438; Manufacturer (none) -> Boom Precision Elec; Mfg part no. (none) -> x2
Connections:
- net +5V: now also JP17.2 (C); no longer D14.1 (K), D15.1 (K)
- net EN: now also C28.1
- net GND: now also C28.2
- net VUSB: now also D15.2 (A)
- new net: D14.1 (K), JP17.1 (A)
- new net: D15.1 (K), JP17.3 (B)
Other:
- moved on the sheet: D15

Commit message: Changed AUX1 connector symbol
Parts:
- J15: symbol Connector_Generic:Conn_02x04_Counter_Clockwise -> Connector_Generic:Conn_02x04_Odd_Even
Changed lines of the file:
@@
 Reset switch
 $Comp
-L Connector_Generic:Conn_02x04_Counter_Clockwise J15
+L Connector_Generic:Conn_02x04_Odd_Even J15
 U 1 1 5C6AAFFE
 P 6800 9250
@@
 L power:+5V #PWR0160
 U 1 1 5C6BF357
-P 6450 9150
-F 0 "#PWR0160" H 6450 9000 50  0001 C CNN
-F 1 "+5V" H 6465 9323 50  0000 C CNN
-F 2 "" H 6450 9150 50  0001 C CNN
-F 3 "" H 6450 9150 50  0001 C CNN
-	1    6450 9150
+P 6600 9150
+F 0 "#PWR0160" H 6600 9000 50  0001 C CNN
+F 1 "+5V" H 6615 9323 50  0000 C CNN
+F 2 "" H 6600 9150 50  0001 C CNN
+F 3 "" H 6600 9150 50  0001 C CNN
+	1    6600 9150
 	1    0    0    -1
 $EndComp
@@
 L power:GND #PWR0162
 U 1 1 5C6BF511
-P 6600 9450
-F 0 "#PWR0162" H 6600 9200 50  0001 C CNN
-F 1 "GND" V 6605 9277 50  0000 C CNN
-F 2 "" H 6600 9450 50  0001 C CNN
-F 3 "" H 6600 9450 50  0001 C CNN
-	1    6600 9450
+P 6600 9250
+F 0 "#PWR0162" H 6600 9000 50  0001 C CNN
+F 1 "GND" V 6605 9077 50  0000 C CNN
+F 2 "" H 6600 9250 50  0001 C CNN
+F 3 "" H 6600 9250 50  0001 C CNN
+	1    6600 9250
 	0    1    1    0
 $EndComp
-Wire Wire Line
-	6600 9150 6450 9150
 $Comp
 L power:+3.3V #PWR0165
@@
 	1    0    0    -1
 $EndComp
-Wire Wire Line
-	6600 9250 6450 9250
-Wire Wire Line
-	6450 9250 6450 9150
-Connection ~ 6450 9150
-Wire Wire Line
-	6600 9350 6600 9450
-Connection ~ 6600 9450
-NoConn ~ 7100 9250
-NoConn ~ 7100 9450
+NoConn ~ 6600 9350
+NoConn ~ 6600 9450
 Text Label 7000 4150 0    50   ~ 0
 D+
@@
 	8100 3650 8100 3450
 Connection ~ 8100 3450
-Text GLabel 7100 9150 2    50   BiDi ~ 0
+Text GLabel 7100 9450 2    50   BiDi ~ 0
 UART-
 Text GLabel 7100 9350 2    50   BiDi ~ 0
@@
 	4150 3650 4150 3950
 Connection ~ 4150 3950
+$Comp
+L power:+5V #PWR?
+U 1 1 5DEF0F24
+P 7100 9150
+F 0 "#PWR?" H 7100 9000 50  0001 C CNN
+F 1 "+5V" H 7115 9323 50  0000 C CNN
+F 2 "" H 7100 9150 50  0001 C CNN
+F 3 "" H 7100 9150 50  0001 C CNN
+	1    7100 9150
+	1    0    0    -1
+$EndComp
+$Comp
+L power:GND #PWR?
+U 1 1 5DEF1033
+P 7100 9250
+F 0 "#PWR?" H 7100 9000 50  0001 C CNN
+F 1 "GND" V 7105 9077 50  0000 C CNN
+F 2 "" H 7100 9250 50  0001 C CNN
+F 3 "" H 7100 9250 50  0001 C CNN
+	1    7100 9250
+	0    -1   -1   0
+$EndComp
 $EndSCHEMATC
